File: BrainRing_Wireless_Players/BrainRing_Wireless_Players.kicad_sch (KiCad schematic)
At the start: 0 parts

Commit message: upd sch
Parts:
- added D9: SS110, Diode_SMD:D_SMA, symbol Diode:SS14
- added J?: LED Strip, symbol Connector:Conn_01x03_Pin
- added Q1: MMBT2222A, Package_TO_SOT_SMD:SOT-23, symbol Transistor_BJT:MMBT2222A
- added R16: 1k, Resistor_SMD:R_0603_1608Metric, symbol Device:R_Small
- added R?: 300, Resistor_SMD:R_0603_1608Metric, symbol Device:R_Small
- added U19: MLT-8530, .my_Audio:MLT8530, symbol .my_Audio:MLT-8530
- added U?: LGT8F328P_LQFP32, .my_Chip:LGT8F328P_LQFP32, symbol .my_Chip:LGT8F328P_LQFP32
- added U?: NRF24L01_Breakout, RF_Module:nRF24L01_Breakout, symbol RF:NRF24L01_Breakout
Connections:
- new net: D9.2 (A), Q1.3 (C), U19.3 (-LEAD)
- new net: J?.2 (Pin_2), R?.2
- new net: Q1.1 (B), R16.1
- new net: R?.1, U?.16 (7)
- new net +3.3V: U?.2 (VCC)
- new net +5V: D9.1 (K), J?.1 (Pin_1), U19.2 (+LEAD), U?.4 (VCC)
- new net BUTTON: U?.20 (3)
- new net BUZZER_PIN: R16.2, U?.19 (4)
- new net CE: U?.3 (CE), U?.33 (9)
- new net CSN: U?.35 (10), U?.4 (~{CSN})
- new net GND: J?.3 (Pin_3), Q1.2 (E), U?.1 (GND), U?.11 (GND), U?.2 (GND), U?.22 (GND)
- new net MISO: U?.10 (12), U?.7 (MISO)
- new net MOSI: U?.34 (11), U?.6 (MOSI)
- new net SCK: U?.5 (SCK), U?.9 (13)
- no-connect marks 0 -> 20
Other:
- added sheet Power Sheet (Power Sheet.kicad_sch)
- note added: "BUZZER"
- note added: "NRF24L01"
