File: pcb/BrainRing_Wireless_Admin/BrainRing_Wireless_Admin.kicad_sch (KiCad schematic)
At the start: 0 parts

Commit message: upd2.0
Parts:
- added D1: SS110, Diode_SMD:D_SMA, symbol Diode:SS14
- added H1, H2: MountingHole, MountingHole:MountingHole_2.2mm_M2, symbol Mechanical:MountingHole
- added J1: Butt+WS2812b, Connector_JST:JST_EH_B4B-EH-A_1x04_P2.50mm_Vertical, symbol Connector:Conn_01x04_Pin
- added Q1: MMBT2222A, Package_TO_SOT_SMD:SOT-23, symbol Transistor_BJT:MMBT2222A
- added R1: 300, Resistor_SMD:R_0603_1608Metric, symbol Device:R_Small
- added R2: 1k, Resistor_SMD:R_0603_1608Metric, symbol Device:R_Small
- added TP1, TP2: Jumper, Connector_PinHeader_2.54mm:PinHeader_1x01_P2.54mm_Vertical, symbol Connector:TestPoint
- added U1: LGT8F328P_LQFP32, .my_Chip:LGT8F328P_LQFP32, symbol .my_Chip:LGT8F328P_LQFP32
- added U2: NRF24L01+PA+LNA, .my_RF:nRF24L01+PA+LNA_Breakout, symbol .my_RF:NRF24L01+PA+LNA
- added U3: MLT-8530, .my_Audio:MLT8530, symbol .my_Audio:MLT-8530
Connections:
- new net: D1.2 (A), Q1.3 (C), U3.3 (-LEAD)
- new net: Q1.1 (B), R2.1
- new net: R1.1, U1.19 (4)
- new net: J1.1 (Pin_1), R1.2
- new net +3.3V: TP1.1, TP2.1, U2.2 (VCC)
- new net +5V: D1.1 (K), J1.3 (Pin_3), U1.4 (VCC), U3.2 (+LEAD)
- new net BUTTON: J1.2 (Pin_2), U1.20 (3)
- new net BUZZER_PIN: R2.2, U1.21 (2)
- new net CE: U1.32 (8), U2.3 (CE)
- new net CSN: U1.33 (9), U2.4 (~{CSN})
- new net GND: J1.4 (Pin_4), Q1.2 (E), U1.2 (GND), U1.22 (GND), U2.1 (GND)
- new net MISO: U1.10 (12), U2.7 (MISO)
- new net MOSI: U1.34 (11), U2.6 (MOSI)
- new net SCK: U1.9 (13), U2.5 (SCK)
- no-connect marks 0 -> 31
Other:
- added sheet Power Sheet (Power Sheet.kicad_sch)
- note added: "BUZZER"
- note added: "NRF24L01"
