File: pcb/BrainRing_Wireless_Admin/BrainRing_Wireless_Admin.kicad_pcb (KiCad board)
At the start: 2 copper layers, 68 x 79 mm, 35 parts, among them J1 Butt+WS2812b, J2 USB_C_Receptacle_PowerOnly_6P, Q1 MMBT2222A, SW1 SS12D11G5, U1 LGT8F328P_LQFP32, U2 NRF24L01+PA+LNA, U3 MLT-8530, U4 IP5305, U5 AMS1117-3.3

Commit message: Refactor firmware: fair first-press detection, single player firmware, animations
- Shared protocol/radio config (include/brainring.h) and non-blocking melody player (include/melody.h)
- Admin: timestamp-based winner resolution with 30 ms decision window, reject pre-reset presses,
  fresh ACK payloads, press/reset sound and LED indication, idle breathing
- Players: one firmware for all boards, ID/color stored in EEPROM with on-device color menu,
  reliable press delivery with per-ID retry delays, link-loss detection,
  strip + button LED (PWM) animations, 3 random win melodies and a lose melody
- Admin case generator, print files and PCB updates

Co-Authored-By: Claude Opus 5.5 <noreply@anthropic.com>
Parts:
- added H1: MountingHole, MountingHole:MountingHole_3.2mm_M3, F.Cu at (176.0, 69.0)
- added H4: MountingHole, MountingHole:MountingHole_2.2mm_M2, F.Cu at (216.1, 128.0)
- added Q2: AO3400A, Package_TO_SOT_SMD:SOT-23, B.Cu at (175.8, 108.6)
- added R7: 100, Resistor_SMD:R_0603_1608Metric, B.Cu at (173.6, 104.0)
- added R8: 100k, Resistor_SMD:R_0603_1608Metric, B.Cu at (177.4, 112.4)
- added R9: 47, Resistor_SMD:R_1206_3216Metric, B.Cu at (178.0, 104.6)
- H2: footprint MountingHole:MountingHole_2.2mm_M2 -> MountingHole:MountingHole_3.2mm_M3
- moved H3 40.1 mm to (216.1, 68.5)
- moved U2 29.2 mm to (206.0, 104.8)
- moved TP1 23.5 mm to (195.6, 100.0)
- moved TP2 14.5 mm to (200.6, 110.0)
- moved C8 13.1 mm to (200.1, 99.0), turned to 90 degrees
- moved C9 12.3 mm to (197.9, 99.0), turned to 90 degrees
- moved R2 0.55 mm to (216.9, 103.3)
- renumbered H1 to H3
Connections:
- U1 pad 32: /CE -> unconnected-(U1-8-Pad32)
- U1 pad 5: unconnected-(U1-A3-Pad5) -> /KEEPALIVE
- U1 pad 8: unconnected-(U1-A0-Pad8) -> /CE
Routing:
- net /CE: track 15.6 -> 111.9 mm
- net /MOSI: track 37.3 -> 58.9 mm
- net GND: track 6.47 -> 28.0 mm
- net /CSN: track 16.7 -> 38.0 mm
- net /MISO: track 58.2 -> 75.7 mm
- net /SCK: track 76.1 -> 90.3 mm
- net Net-(Q2-G): track 0.00 -> 12.1 mm
- net /KEEPALIVE: track 0.00 -> 11.8 mm
- net +3.3V: track 22.6 -> 17.1 mm
- net Net-(Q2-D): track 0.00 -> 3.30 mm
- net /BUZZER_PIN: track 51.8 -> 52.3 mm
- net Net-(Q1-B): track 2.20 -> 1.65 mm
Other:
- board text added: "27.10.2026 Rev. 2.1"
- board text removed: "16.04.2026 Rev. 2.0"
