File: pcb/BrainRing_Wireless_Players/BrainRing_Wireless_Players.kicad_sch (KiCad schematic)
At the start: 8 parts, among them Q1 MMBT2222A, U19 MLT-8530

Commit message: upd2.0
Parts:
- added H1, H2: MountingHole, MountingHole:MountingHole_2.2mm_M2, symbol Mechanical:MountingHole
- added J2: Arcade_Button, Connector_JST:JST_EH_B4B-EH-A_1x04_P2.50mm_Vertical, symbol Connector:Conn_01x04_Pin
- added J3, J4: Jumper, Connector_PinHeader_2.54mm:PinHeader_1x01_P2.54mm_Vertical, symbol Connector:Conn_01x01_Pin
- added R2: 100, Resistor_SMD:R_0603_1608Metric, symbol Device:R_Small
- J1: renamed from J?; value LED Strip -> LED_Strip; footprint (none) -> Connector_JST:JST_EH_B3B-EH-A_1x03_P2.50mm_Vertical
- gave numbers to parts that had none: 3
- renumbered D9 to D1, R16 to R3, U19 to U3
Connections:
- net +5V: now also J1.2 (Pin_2); no longer J1.1 (Pin_1)
- net BUTTON: now also J2.2 (Pin_2)
- net BUZZER_PIN: now also U1.21 (2); no longer U1.19 (4)
- net CE: now also U1.32 (8); no longer U1.33 (9)
- net CSN: now also U1.33 (9); no longer U1.35 (10)
- net GND: now also J1.1 (Pin_1), U3.1 (DUMMY_PAD_1), U3.4 (DUMMY_PAD_2), J2.3 (Pin_3), J2.4 (Pin_4), J3.1 (Pin_1), J4.1 (Pin_1); no longer J1.3 (Pin_3), U1.11 (GND)
- net at R1.2: now also J1.3 (Pin_3); no longer J1.2 (Pin_2)
- net at U1.16 (7): no longer R1.1
- net at U1.17 (6): now also R2.1
- new net: R1.1, U1.19 (4)
- new net BUT_LED: J2.1 (Pin_1), R2.2
- no-connect marks 20 -> 28
Other:
- moved on the sheet: J1, R1
