File: pcb/BrainRing_Wireless_Players/Power Sheet.kicad_sch (KiCad schematic)
At the start: 23 parts, among them U2 AMS1117-3.3

Commit message: upd2.0
Parts:
- BT1: renamed from BT?; footprint BH-18650-PC:BAT_BH-18650-PC -> .my_Connector:BAT_BH-18650-PC
- D2, D3, D4, D5: renamed from D?; footprint (none) -> LED_SMD:LED_0805_2012Metric
- J5: renamed from J?; footprint (none) -> Connector_USB:USB_C_Receptacle_HRO_TYPE-C-31-M-17
- L1: renamed from L?; footprint (none) -> Inductor_SMD:L_APV_APH0630
- gave numbers to parts that had none: 10
- renumbered C1 to C2, C2 to C6, C3 to C8, R11 to R4, R12 to R5, U2 to U5
Connections:
- net at C4.1, C7.1, U4.8 (Vout): now also SW1.3 (C); no longer SW1.1 (A)
