File: pcb/BrainRing_Wireless_Players/BrainRing_Wireless_Players.kicad_pcb (KiCad board)
At the start: 2 copper layers, 80 x 58 mm, 37 parts, among them J1 LED_Strip, J2 Arcade_Button, J3 Jumper, J4 Jumper, J5 USB_C_Receptacle_PowerOnly_6P, Q1 MMBT2222A, SW1 SS12D11G5, U1 LGT8F328P_LQFP32, U2 NRF24L01_Breakout, U3 MLT-8530, U4 IP5305, U5 AMS1117-3.3

Commit message: Players board Rev. 2.1: IP5305 keep-alive load
- Schematic/PCB: AO3400A (Q2) + 47 Ohm load (R10), gate R8 100 / R9 100k,
  driven from U1 A3 — same circuit as the Admin board. Placed on B.Cu
  under the MCU module; main parts and case-related positions unchanged.
- GND via enlarged to 1.6/0.8 mm for a top-side wire jumper to U1 GND.
- Player firmware: 300 ms pulse every 15 s on A3 so IP5305 doesn't shut
  the 5V output down at light load.
- Regenerated laser-printer sheets (B.Cu, mirrored F.Silkscreen).

Co-Authored-By: Claude Opus 5.5 <noreply@anthropic.com>
Parts:
- added Q2: AO3400A, Package_TO_SOT_SMD:SOT-23, B.Cu at (202.8, 66.6)
- added R10: 47, Resistor_SMD:R_1206_3216Metric, B.Cu at (201.4, 63.5)
- added R8: 100, Resistor_SMD:R_0603_1608Metric, B.Cu at (204.6, 64.0)
- added R9: 100k, Resistor_SMD:R_0603_1608Metric, B.Cu at (203.0, 69.9)
Connections:
- U1 pad 5: unconnected-(U1-A3-Pad5) -> /KEEPALIVE
Routing:
- net GND: track 0.07 -> 8.35 mm, vias 0 -> 1
- net Net-(Q2-G): track 0.00 -> 5.41 mm
- net /KEEPALIVE: track 0.00 -> 4.30 mm
- net +5V: track 80.4 -> 84.1 mm
- net Net-(Q2-D): track 0.00 -> 2.16 mm
Other:
- board text added: "29.10.2026"
- board text added: "Jumper2"
- board text added: "Rev. 2.1"
- board text removed: "16.04.2026"
- board text removed: "Rev. 2.0"
